File: Antlia/Antlia.kicad_sch (KiCad schematic)
At the start: 0 parts

Commit message: Add initial KiCad design for Antlia MEMS microphone breakout
This commit introduces the schematic and PCB layout for the Antlia project, featuring the Infineon IM73D122 MEMS microphone.

The design includes:
*   Schematic capture with the microphone (U1), a decoupling capacitor (C1), a pull-up resistor (R1), and a 4-pin header (J1).
*   PCB layout with corresponding component placement, routing, ground pours, and mounting holes.
*   Custom symbol, footprint, and 3D model for the IM73D122.
*   Project configuration and initial fabrication options.
Parts:
- added C1: 100nF, Capacitor_SMD:C_0603_1608Metric, symbol Device:C
- added H1, H2: MountingHole, MountingHole:MountingHole_2.2mm_M2, symbol Mechanical:MountingHole
- added J1: Conn_01x04_Pin, Connector_PinHeader_2.54mm:PinHeader_1x04_P2.54mm_Vertical, symbol Connector:Conn_01x04_Pin
- added R1: 100, Capacitor_SMD:C_0603_1608Metric, symbol Device:R
- added U1: IM73D122V01XTMA1, Sensor_Audio:Infineon_PG-LLGA-5-2, symbol 2026-09-22_11-15-35:IM73D122V01XTMA1
Connections:
- new net: R1.1, U1.1 (DATA)
- new net +1V8: C1.1, J1.1 (Pin_1), U1.2 (VDD)
- new net GND: C1.2, J1.2 (Pin_2), U1.4 (LR), U1.5 (GND)
- new net MIC_CLOCK: J1.4 (Pin_4), U1.3 (CLOCK)
- new net MIC_DATA: J1.3 (Pin_3), R1.2
